File: FET_Half_Bridge.kicad_sch (KiCad schematic)
At the start: 13 parts, among them Q1 NMOS, Q2 NMOS

Commit message: start layout
Connections:
- net GATE_H_RAW: now reaches D4.2 (A), Q1.1 (G), R21.2
- net GATE_L_RAW: now reaches D5.2 (A), D6.1 (K), Q2.1 (G), R22.2
Changed lines of the file:
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@@
+		)
+	)
+	(label "GATE_L_RAW"
+		(at 125.73 106.68 0)
+		(effects
+			(font
+				(size 1.27 1.27)
+			)
+			(justify left bottom)
+		)
+	)
+	(label "GATE_H_RAW"
+		(at 125.73 85.09 0)
+		(effects
+			(font
+				(size 1.27 1.27)
+			)
+			(justify left bottom)
 		)
 	)

Commit message: placed more components
Parts:
- removed C24, C25: 4.7uF/50V, hn_lib:hn_C_1206, symbol Device:C
- renumbered C26 to C24, C27 to C25
