File: Microcontroller.kicad_sch (KiCad schematic)
At the start: 43 parts, among them U1 TCAN334G, U2 STM32G474CETx, U3 AS5047D, Y1 24MHz/CL=10pF

Commit message: start layout
Parts:
- renumbered L2 to L1
Changed lines of the file:
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@@
 		(dnp no)
 		(fields_autoplaced yes)
-		(property "Reference" "L2"
+		(property "Reference" "L1"
 			(at 80.01 168.91 90)
 			(effects
@@
 			(project ""
 				(path "/c8b2ce32-1e5b-45e4-8f0b-d70c39b97a8d/7a6505cb-5d4b-46b8-92a2-882c1defdbef"
-					(reference "L2")
+					(reference "L1")
 					(unit 1)
 				)

Commit message: placed more components
Connections:
- net GNDA is gone; now on net GND: C11.2, C12.2, C13.2, C14.2, U2.19 (VSSA)
Changed lines of the file:
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@@
 	)
 	(junction
+		(at 165.1 127)
+		(diameter 0)
+		(color 0 0 0 0)
+	)
+	(junction
 		(at 50.8 48.26)
 		(diameter 0)
@@
 	(wire
 		(pts
+			(xy 165.1 127) (xy 167.64 127)
+		)
+		(stroke
+			(width 0)
+			(type default)
+		)
+	)
+	(wire
+		(pts
 			(xy 165.1 40.64) (xy 165.1 41.91)
 		)
@@
 	)
 	(symbol
+		(lib_id "power:GND")
+		(at 99.06 186.69 0)
+		(unit 1)
+		(exclude_from_sim no)
+		(in_bom yes)
+		(on_board yes)
+		(dnp no)
+		(fields_autoplaced yes)
+		(property "Reference" "#PWR018"
+			(at 99.06 193.04 0)
+			(effects
+				(font
+					(size 1.27 1.27)
+				)
+				(hide yes)
+			)
+		)
+		(property "Value" "GND"
+			(at 99.06 191.77 0)
+			(effects
+				(font
+					(size 1.27 1.27)
+				)
+			)
+		)
+		(property "Footprint" ""
+			(at 99.06 186.69 0)
+			(effects
+				(font
+					(size 1.27 1.27)
+				)
+				(hide yes)
+			)
+		)
+		(property "Datasheet" ""
+			(at 99.06 186.69 0)
+			(effects
+				(font
+					(size 1.27 1.27)
+				)
+				(hide yes)
+			)
+		)
+		(property "Description" ""
+			(at 99.06 186.69 0)
+			(effects
+				(font
+					(size 1.27 1.27)
+				)
+			)
+		)
+		(pin "1"
+		)
+		(instances
+			(project "spinor-r2a"
+				(path "/c8b2ce32-1e5b-45e4-8f0b-d70c39b97a8d/7a6505cb-5d4b-46b8-92a2-882c1defdbef"
+					(reference "#PWR018")
+					(unit 1)
+				)
+			)
+		)
+	)
+	(symbol
 		(lib_id "Device:R_US")
 		(at 39.37 82.55 270)
@@
 					(unit 1)
 				)
-			)
-		)
-	)
-	(symbol
-		(lib_name "GNDA_1")
-		(lib_id "power:GNDA")
-		(at 99.06 186.69 0)
-		(unit 1)
-		(exclude_from_sim no)
-		(in_bom yes)
-		(on_board yes)
-		(dnp no)
-		(fields_autoplaced yes)
-		(property "Reference" "#PWR024"
-			(at 99.06 193.04 0)
-			(effects
-				(font
-					(size 1.27 1.27)
-				)
-				(hide yes)
-			)
-		)
-		(property "Value" "GNDA"
-			(at 99.06 191.77 0)
-			(effects
-				(font
-					(size 1.27 1.27)
-				)
-			)
-		)
-		(property "Footprint" ""
-			(at 99.06 186.69 0)
-			(effects
-				(font
-					(size 1.27 1.27)
-				)
-				(hide yes)
-			)
-		)
-		(property "Datasheet" ""
-			(at 99.06 186.69 0)
-			(effects
-				(font
-					(size 1.27 1.27)
-				)
-				(hide yes)
-			)
-		)
-		(property "Description" "Power symbol creates a global label with name \"GNDA\" , analog ground"
-			(at 99.06 186.69 0)
-			(effects
-				(font
-					(size 1.27 1.27)
-				)
-				(hide yes)
-			)
-		)
-		(pin "1"
-		)
-		(instances
-			(project "spinor-r2a"
-				(path "/c8b2ce32-1e5b-45e4-8f0b-d70c39b97a8d/7a6505cb-5d4b-46b8-92a2-882c1defdbef"
-					(reference "#PWR024")
-					(unit 1)
-				)
-			)
-		)
-	)
-	(symbol
-		(lib_name "GNDA_1")
-		(lib_id "power:GNDA")
-		(at 167.64 127 0)
-		(unit 1)
-		(exclude_from_sim no)
-		(in_bom yes)
-		(on_board yes)
-		(dnp no)
-		(fields_autoplaced yes)
-		(property "Reference" "#PWR018"
-			(at 167.64 133.35 0)
-			(effects
-				(font
-					(size 1.27 1.27)
-				)
-				(hide yes)
-			)
-		)
-		(property "Value" "GNDA"
-			(at 167.64 132.08 0)
-			(effects
-				(font
-					(size 1.27 1.27)
-				)
-			)
-		)
-		(property "Footprint" ""
-			(at 167.64 127 0)
-			(effects
-				(font
-					(size 1.27 1.27)
-				)
-				(hide yes)
-			)
-		)
-		(property "Datasheet" ""
-			(at 167.64 127 0)
-			(effects
-				(font
-					(size 1.27 1.27)
-				)
-				(hide yes)
-			)
-		)
-		(property "Description" "Power symbol creates a global label with name \"GNDA\" , analog ground"
-			(at 167.64 127 0)
-			(effects
-				(font
-					(size 1.27 1.27)
-				)
-				(hide yes)
-			)
-		)
-		(pin "1"
-		)
-		(instances
-			(project "spinor-r2a"
-				(path "/c8b2ce32-1e5b-45e4-8f0b-d70c39b97a8d/7a6505cb-5d4b-46b8-92a2-882c1defdbef"
-					(reference "#PWR018")
-					(unit 1)
-				)

Commit message: ok
Parts:
- removed C13, C4: 100nF/6.3V, hn_lib:hn_C_0402, symbol Device:C
Other:
- moved on the sheet: C12

Commit message: done routing!
Parts:
- removed J3, J4: ~, Connector_PinHeader_1.27mm:PinHeader_1x04_P1.27mm_Vertical, symbol Connector_Generic:Conn_01x04
- removed R7, R8: 100R, hn_lib:hn_R_0402, symbol Device:R_US
- added J9: Conn_01x05, Connector_PinHeader_2.54mm:PinHeader_1x05_P2.54mm_Vertical, symbol Connector_Generic:Conn_01x05
- added TP13: ~, Connector_PinHeader_1.00mm:PinHeader_1x01_P1.00mm_Vertical, symbol Connector:TestPoint
Connections:
- net DEBUG_NRST: now also J9.2 (Pin_2)
- net DEBUG_SWCLK: now also J9.3 (Pin_3)
- net DEBUG_SWDIO: now also J9.4 (Pin_4)
- net DEBUG_VTGT: now also J9.5 (Pin_5)
- net DRV_IA: now also U2.16 (PB0); no longer U2.17 (PB1)
- net DRV_IB: now also U2.17 (PB1); no longer U2.18 (PB2)
- net DRV_IC: now also U2.18 (PB2); no longer U2.16 (PB0)
- net GND: now also J9.1 (Pin_1); no longer D1.3 (A), J1.1 (Pin_1), J2.1 (Pin_1)
- net USART1_TX: now also TP13.1
- net CANH renamed CAN_P
- net CANL renamed CAN_N
- net USART1_RX: no longer names the net of U2.44 (PB7)
- new net GNDPWR: D1.3 (A), J1.1 (Pin_1), J2.1 (Pin_1)
Other:
- note added: "Power GND used for TVS and CAN connector GND from routing considerations"
- moved on the sheet: R6
