File: Power_Supply.kicad_sch (KiCad schematic)
At the start: 17 parts, among them U5 TPS560430X3FDBVR

Commit message: start layout
Parts:
- removed C37: 100uF/63V, hn_lib:hn_C_Kemet_A768MS, symbol Device:C_Polarized
- J9: footprint hn_lib:hn_AMASS_XT30PW-F -> hn_lib:hn_AMASS_XT30PW-M; part Amass XT30-PW-F -> Amass XT30-PW-M
- renumbered L3 to L2, L1 to L3

Commit message: placed more components
Parts:
- added C38, C39, C40, C41, C42, C43, C44, C45, C46, C47, C48, C49, C52, C53, C54, C55: 4.7uF/50V, hn_lib:hn_C_1206, symbol Device:C
- added NT1: NetTie_2, symbol Device:NetTie_2
- renumbered C36 to C30, C38 to C31, C39 to C32, C40 to C33, C41 to C34, C42 to C35, C43 to C36, C44 to C37
Connections:
- net GND: now also NT1.2; no longer C30.2, C31.2, D13.2 (A), J8.1 (Pin_1), J9.1 (Pin_1)
- net VBUS: now also C38.1, C39.1, C40.1, C41.1, C42.1, C43.1, C44.1, C45.1, C46.1, C47.1, C48.1, C49.1, C52.1, C53.1, C54.1, C55.1
- new net GNDPWR: C30.2, C31.2, C38.2, C39.2, C40.2, C41.2, C42.2, C43.2, C44.2, C45.2, C46.2, C47.2, C48.2, C49.2, C52.2, C53.2, C54.2, C55.2, D13.2 (A), J8.1 (Pin_1), J9.1 (Pin_1), NT1.1
Other:
- note added: "Tie grounds together at one point near 3V3 reg"
- note removed: "Tie grounds together at one point"
- moved on the sheet: C31

Commit message: layout driver and 3v3 buck
Parts:
- removed C35: 100nF/50V, hn_lib:hn_C_0603, symbol Device:C
- removed L2: FB/120R@100MHz, hn_lib:hn_R_0805, symbol Device:L
Connections:
- net VBUS: now also C36.1, C37.1, U5.4 (EN), U5.5 (VIN)
- net 3V3_BUCK_CP: now reaches C33.2, U5.1 (CB)
Other:
- note added: "EN pin tied to Vin. UVLO at 3.45V in event of power cut during motor spin: MCU fw detects low Vin and switches on all 3 low-side FETs if Vin keeps falling, it will hit 8V UVLO of DRV chip which disables all FETs. hopefully motor has by then stopped spinning. if not, body diodes can take the heat. at Vin ~5V, fw is set up to halt. brownout detector is also used to induce a reset in glitchy cases. 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"
- note removed: "EN pin thresholds: rising 1.23V, falling 1.1V 470k upper 100k lower leads to 7V turn-on and 6.3 turn-off thresholds"
- note removed: "EN pin tied to Vin. UVLO at 3.45V in event of power cut during motor spin: MCU fw detects low Vin and switches on all 3 low-side FETs if Vin keeps falling, it will hit 8V UVLO of DRV chip which disables all FETs. hopefully motor has by then stopped spinning. if not, body diodes can take the heat. at Vin ~5V, fw is set up to halt. brownout detector is also used to induce a reset in glitchy cases."
Changed lines of the file:
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@@
 		)
 	)
-	(text "EN pin thresholds: rising 1.23V, falling 1.1V\n470k upper 100k lower leads to 7V turn-on and 6.3 turn-off thresholds"
-		(exclude_from_sim no)
-		(at 359.664 87.376 0)
-		(effects
-			(font
-				(size 1.27 1.27)
-			)
-		)
-	)
 	(text "Follow datasheet 9.2.2 Detailed design procedure\n\ninductor selection\n\nLmin = (Vin,max - Vout) / (Iout,min * Kind) * Vout / (Vin,max * fsw)\nfsw = 1.1MHz (fixed for this part)\nVout = 3.3V\nVin,max = 25.2V\nKind = 20-60% (use 0.6)\nIout,min = 150mA (use max or answer is unreasonably large)\n=> Lmin = 43.5uH => use 47uH\ninductor needs to handle 150mA load + 50mA ripple.\nChoose ~500mA rating, saturation a bit higher.\n\nDelta I_L = Vout * (Vin,max-Vout)/(Vin,max * L * f_sw) = 55mA\n\noutput capacitor selection\nESR ripple = Delta I_L * ESR = 55mA * = \nCharging ripple = Delta I_L / (8*f_sw * C_out) = 0.6mV\nLoad step stability: require\nC_out > 4 * (load step) / (f_sw * Delta V_out) = 2uF\nfor load step = 150mA, Delta V_out = 250mV\n\ninput capacitor\n2.2uF/50V Low ESR\n\nbootstrap cap\n100nF/16V\n\n"
 		(exclude_from_sim no)
@@
 		)
 	)
-	(text "EN pin tied to Vin. UVLO at 3.45V\nin event of power cut during motor spin:\nMCU fw detects low Vin and switches on all 3 low-side FETs\nif Vin keeps falling, it will hit 8V UVLO of DRV chip\nwhich disables all FETs. hopefully motor has by then stopped spinning.\nif not, body diodes can take the heat.\nat Vin ~5V, fw is set up to halt.\nbrownout detector is also used to induce a reset in glitchy cases."
+	(text "EN pin tied to Vin. UVLO at 3.45V\nin event of power cut during motor spin:\nMCU fw detects low Vin and switches on all 3 low-side FETs\nif Vin keeps falling, it will hit 8V UVLO of DRV chip\nwhich disables all FETs. hopefully motor has by then stopped spinning.\nif not, body diodes can take the heat.\nat Vin ~5V, fw is set up to halt.\nbrownout detector is also used to induce a reset in glitchy cases.\nat 3.45V, regulator shuts off"
 		(exclude_from_sim no)
 		(at 356.108 74.93 0)
@@
 	)
 	(junction
-		(at 71.12 148.59)
-		(diameter 0)
-		(color 0 0 0 0)
-	)
-	(junction
 		(at 176.53 166.37)
 		(diameter 0)
@@
 	)
 	(junction
-		(at 38.1 123.19)
-		(diameter 0)
-		(color 0 0 0 0)
-	)
-	(junction
 		(at 224.79 48.26)
 		(diameter 0)
@@
 	(wire
 		(pts
-			(xy 38.1 123.19) (xy 38.1 130.81)
-		)
-		(stroke
-			(width 0)
-			(type default)
-		)
-	)
-	(wire
-		(pts
 			(xy 87.63 123.19) (xy 116.84 123.19)
 		)
@@
 	(wire
 		(pts
-			(xy 38.1 148.59) (xy 71.12 148.59)
-		)
-		(stroke
-			(width 0)
-			(type default)
-		)
-	)
-	(wire
-		(pts
 			(xy 86.36 40.64) (xy 86.36 45.72)
 		)
@@
 	(wire
 		(pts
-			(xy 53.34 123.19) (xy 71.12 123.19)
-		)
-		(stroke
-			(width 0)
-			(type default)
-		)
-	)
-	(wire
-		(pts
 			(xy 73.66 77.47) (xy 73.66 92.71)
 		)
@@
 	(wire
 		(pts
-			(xy 27.94 123.19) (xy 38.1 123.19)
+			(xy 27.94 123.19) (xy 71.12 123.19)
 		)
 		(stroke
@@
 	(wire
 		(pts
-			(xy 38.1 138.43) (xy 38.1 148.59)
-		)
-		(stroke
-			(width 0)
-			(type default)
-		)
-	)
-	(wire
-		(pts
 			(xy 246.38 180.34) (xy 246.38 177.8)
 		)
@@
 	(wire
 		(pts
-			(xy 38.1 123.19) (xy 45.72 123.19)
+			(xy 81.28 179.07) (xy 64.77 179.07)
 		)
 		(stroke
@@
 	(wire
 		(pts
-			(xy 81.28 179.07) (xy 64.77 179.07)
+			(xy 81.28 168.91) (xy 81.28 166.37)
 		)
 		(stroke
@@
 		)
 	)
-	(wire
-		(pts
-			(xy 81.28 168.91) (xy 81.28 166.37)
+	(label "VBUS_FILT"
+		(at 64.77 123.19 0)
+		(effects
+			(font
+				(size 1.27 1.27)
+			)
+			(justify left bottom)
 		)
-		(stroke
-			(width 0)
-			(type default)
+	)
+	(label "3V3_BUCK_CP"
+		(at 171.45 130.81 0)
+		(effects
+			(font
+				(size 1.27 1.27)
+			)
+			(justify left bottom)
 		)
 	)
@@
 	)
 	(symbol
-		(lib_id "Device:C")
-		(at 38.1 134.62 0)
-		(unit 1)
-		(exclude_from_sim no)
-		(in_bom yes)
-		(on_board yes)
-		(dnp no)
-		(fields_autoplaced yes)
-		(property "Reference" "C35"
-			(at 41.91 133.3499 0)
-			(effects
-				(font
-					(size 1.27 1.27)
-				)
-				(justify left)
-			)
-		)
-		(property "Value" "100nF/50V"
-			(at 41.91 135.8899 0)
-			(effects
-				(font
-					(size 1.27 1.27)
-				)
-				(justify left)
-			)
-		)
-		(property "Footprint" "hn_lib:hn_C_0603"
-			(at 39.0652 138.43 0)
-			(effects
-				(font
-					(size 1.27 1.27)
-				)
-				(hide yes)
-			)
-		)
-		(property "Datasheet" "~"
-			(at 38.1 134.62 0)
-			(effects
-				(font
-					(size 1.27 1.27)
-				)
-				(hide yes)
-			)
-		)
-		(property "Description" "Unpolarized capacitor"
-			(at 38.1 134.62 0)
-			(effects
-				(font
-					(size 1.27 1.27)
-				)
-				(hide yes)
-			)
-		)
-		(property "part" "Murata GCJ188R71H104KA12D"
-			(at 38.1 134.62 0)
-			(effects
-				(font
-					(size 1.27 1.27)
-				)
-				(hide yes)
-			)
-		)
-		(pin "2"
-		)
-		(pin "1"
-		)
-		(instances
-			(project "spinor-r2a"
-				(path "/c8b2ce32-1e5b-45e4-8f0b-d70c39b97a8d/fc1e53d0-a8df-47e2-96b1-1922b9156006"
-					(reference "C35")
-					(unit 1)
-				)
-			)
-		)
-	)
-	(symbol
 		(lib_id "power:GND")
 		(at 214.63 62.23 0)
@@
 					(unit 1)
 				)
-			)
-		)
-	)
-	(symbol
-		(lib_id "Device:L")
-		(at 49.53 123.19 90)
-		(unit 1)
-		(exclude_from_sim no)
-		(in_bom yes)
-		(on_board yes)
-		(dnp no)
-		(fields_autoplaced yes)
-		(property "Reference" "L2"
-			(at 49.53 118.11 90)
-			(effects
-				(font
-					(size 1.27 1.27)
-				)
-			)
-		)
-		(property "Value" "FB/120R@100MHz"
-			(at 49.53 120.65 90)
-			(effects
-				(font
-					(size 1.27 1.27)
-				)
-			)
-		)
-		(property "Footprint" "hn_lib:hn_R_0805"
-			(at 49.53 123.19 0)
-			(effects
-				(font
-					(size 1.27 1.27)
-				)
-				(hide yes)
-			)
-		)
-		(property "Datasheet" "~"
-			(at 49.53 123.19 0)
-			(effects
-				(font
-					(size 1.27 1.27)
-				)
-				(hide yes)
-			)
-		)
-		(property "Description" "Inductor"
-			(at 49.53 123.19 0)
-			(effects
-				(font
-					(size 1.27 1.27)
-				)
-				(hide yes)
-			)
-		)
-		(property "part" "Laird SiLaird HI0805O121R-10"
-			(at 49.53 123.19 90)
-			(effects
-				(font
-					(size 1.27 1.27)
-				)
-				(hide yes)
-			)
-		)
-		(pin "2"
-		)
-		(pin "1"
-		)
-		(instances
-			(project "spinor-r2a"
-				(path "/c8b2ce32-1e5b-45e4-8f0b-d70c39b97a8d/fc1e53d0-a8df-47e2-96b1-1922b9156006"
-					(reference "L2")
-					(unit 1)
-				)

Commit message: done routing!
Parts:
- removed J9: ~, hn_lib:hn_AMASS_XT30PW-M, symbol Connector_Generic:Conn_01x02
- removed NT1: NetTie_2, symbol Device:NetTie_2
- added C4: 100uF/63V, hn_lib:hn_C_Kemet_A768MS, symbol Device:C_Polarized
- added C58, C59, C60, C61, C62, C63, C64, C65, C66, C67, C68, C69: 4.7uF/50V, hn_lib:hn_C_1206, symbol Device:C
Connections:
- net GNDPWR is gone; now on net GND: C30.2, C31.2, C38.2, C39.2, C40.2, C41.2, C42.2, C43.2, C44.2, C45.2, C46.2, C47.2, C48.2, C49.2, C52.2, C53.2, C54.2, C55.2, D13.2 (A), J8.1 (Pin_1)
- net GND: now also C4.2, C58.2, C59.2, C60.2, C61.2, C62.2, C63.2, C64.2, C65.2, C66.2, C67.2, C68.2, C69.2
- net VBUS: now also C4.1, C58.1, C59.1, C60.1, C61.1, C62.1, C63.1, C64.1, C65.1, C66.1, C67.1, C68.1, C69.1
