File: Thermistors.kicad_sch (KiCad schematic)
At the start: 7 parts

Commit message: placed more components
Parts:
- renumbered C45 to C50, C46 to C51
Connections:
- net GNDA renamed GND
Changed lines of the file:
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@@
 		(dnp no)
 		(fields_autoplaced yes)
-		(property "Reference" "#PWR052"
+		(property "Reference" "#PWR051"
 			(at 135.89 73.66 0)
 			(effects
@@
 			(project "spinor-r2a"
 				(path "/c8b2ce32-1e5b-45e4-8f0b-d70c39b97a8d/178e97e8-5a17-4ecc-b78e-a0f8597739a5"
-					(reference "#PWR052")
-					(unit 1)
-				)
-			)
-		)
-	)
-	(symbol
-		(lib_id "power:GNDA")
-		(at 135.89 100.33 0)
-		(unit 1)
-		(exclude_from_sim no)
-		(in_bom yes)
-		(on_board yes)
-		(dnp no)
-		(fields_autoplaced yes)
-		(property "Reference" "#PWR054"
-			(at 135.89 106.68 0)
-			(effects
-				(font
-					(size 1.27 1.27)
-				)
-				(hide yes)
-			)
-		)
-		(property "Value" "GNDA"
-			(at 135.89 105.41 0)
-			(effects
-				(font
-					(size 1.27 1.27)
-				)
-			)
-		)
-		(property "Footprint" ""
-			(at 135.89 100.33 0)
-			(effects
-				(font
-					(size 1.27 1.27)
-				)
-				(hide yes)
-			)
-		)
-		(property "Datasheet" ""
-			(at 135.89 100.33 0)
-			(effects
-				(font
-					(size 1.27 1.27)
-				)
-				(hide yes)
-			)
-		)
-		(property "Description" "Power symbol creates a global label with name \"GNDA\" , analog ground"
-			(at 135.89 100.33 0)
-			(effects
-				(font
-					(size 1.27 1.27)
-				)
-				(hide yes)
-			)
-		)
-		(pin "1"
-		)
-		(instances
-			(project ""
-				(path "/c8b2ce32-1e5b-45e4-8f0b-d70c39b97a8d/178e97e8-5a17-4ecc-b78e-a0f8597739a5"
-					(reference "#PWR054")
+					(reference "#PWR051")
 					(unit 1)
 				)
@@
 		(dnp no)
 		(fields_autoplaced yes)
-		(property "Reference" "#PWR053"
+		(property "Reference" "#PWR052"
 			(at 181.61 73.66 0)
 			(effects
@@
 		(property "Description" ""
 			(at 181.61 69.85 0)
+			(effects
+				(font
+					(size 1.27 1.27)
+				)
+			)
+		)
+		(pin "1"
+		)
+		(instances
+			(project "spinor-r2a"
+				(path "/c8b2ce32-1e5b-45e4-8f0b-d70c39b97a8d/178e97e8-5a17-4ecc-b78e-a0f8597739a5"
+					(reference "#PWR052")
+					(unit 1)
+				)
+			)
+		)
+	)
+	(symbol
+		(lib_id "power:GND")
+		(at 181.61 100.33 0)
+		(unit 1)
+		(exclude_from_sim no)
+		(in_bom yes)
+		(on_board yes)
+		(dnp no)
+		(fields_autoplaced yes)
+		(property "Reference" "#PWR053"
+			(at 181.61 106.68 0)
+			(effects
+				(font
+					(size 1.27 1.27)
+				)
+				(hide yes)
+			)
+		)
+		(property "Value" "GND"
+			(at 181.61 105.41 0)
+			(effects
+				(font
+					(size 1.27 1.27)
+				)
+			)
+		)
+		(property "Footprint" ""
+			(at 181.61 100.33 0)
+			(effects
+				(font
+					(size 1.27 1.27)
+				)
+				(hide yes)
+			)
+		)
+		(property "Datasheet" ""
+			(at 181.61 100.33 0)
+			(effects
+				(font
+					(size 1.27 1.27)
+				)
+				(hide yes)
+			)
+		)
+		(property "Description" ""
+			(at 181.61 100.33 0)
 			(effects
 				(font
@@
 		(dnp no)
 		(fields_autoplaced yes)
-		(property "Reference" "C46"
+		(property "Reference" "C51"
 			(at 198.12 90.1699 0)
 			(effects
@@
 			(project "spinor-r2a"
 				(path "/c8b2ce32-1e5b-45e4-8f0b-d70c39b97a8d/178e97e8-5a17-4ecc-b78e-a0f8597739a5"
-					(reference "C46")
-					(unit 1)
-				)
-			)
-		)
-	)
-	(symbol
-		(lib_id "power:GNDA")
-		(at 181.61 100.33 0)
-		(unit 1)
-		(exclude_from_sim no)
-		(in_bom yes)
-		(on_board yes)
-		(dnp no)
-		(fields_autoplaced yes)
-		(property "Reference" "#PWR055"
-			(at 181.61 106.68 0)
-			(effects
-				(font
-					(size 1.27 1.27)
-				)
-				(hide yes)
-			)
-		)
-		(property "Value" "GNDA"
-			(at 181.61 105.41 0)
+					(reference "C51")
+					(unit 1)
+				)
+			)
+		)
+	)
+	(symbol
+		(lib_id "power:GND")
+		(at 135.89 100.33 0)
+		(unit 1)
+		(exclude_from_sim no)
+		(in_bom yes)
+		(on_board yes)
+		(dnp no)
+		(fields_autoplaced yes)
+		(property "Reference" "#PWR054"
+			(at 135.89 106.68 0)
+			(effects
+				(font
+					(size 1.27 1.27)
+				)
+				(hide yes)
+			)
+		)
+		(property "Value" "GND"
+			(at 135.89 105.41 0)
 			(effects
 				(font
@@
 		)
 		(property "Footprint" ""
-			(at 181.61 100.33 0)
+			(at 135.89 100.33 0)
 			(effects
 				(font
@@
 		)
 		(property "Datasheet" ""
-			(at 181.61 100.33 0)
-			(effects
-				(font
-					(size 1.27 1.27)
-				)
-				(hide yes)
-			)
-		)
-		(property "Description" "Power symbol creates a global label with name \"GNDA\" , analog ground"
-			(at 181.61 100.33 0)
-			(effects
-				(font
-					(size 1.27 1.27)
-				)
-				(hide yes)
-			)
-		)
-		(pin "1"
-		)
-		(instances
-			(project "spinor-r2a"
-				(path "/c8b2ce32-1e5b-45e4-8f0b-d70c39b97a8d/178e97e8-5a17-4ecc-b78e-a0f8597739a5"
-					(reference "#PWR055")
+			(at 135.89 100.33 0)
+			(effects
+				(font
+					(size 1.27 1.27)
+				)
+				(hide yes)
+			)
+		)
+		(property "Description" ""
+			(at 135.89 100.33 0)
+			(effects
+				(font
+					(size 1.27 1.27)
+				)
+			)
+		)
+		(pin "1"
+		)
+		(instances
+			(project "spinor-r2a"
+				(path "/c8b2ce32-1e5b-45e4-8f0b-d70c39b97a8d/178e97e8-5a17-4ecc-b78e-a0f8597739a5"
+					(reference "#PWR054")
 					(unit 1)
 				)
@@
 		(dnp no)
 		(fields_autoplaced yes)
-		(property "Reference" "C45"
+		(property "Reference" "C50"
 			(at 153.67 90.1699 0)
 			(effects
@@
 			(project "spinor-r2a"
 				(path "/c8b2ce32-1e5b-45e4-8f0b-d70c39b97a8d/178e97e8-5a17-4ecc-b78e-a0f8597739a5"
-					(reference "C45")
-					(unit 1)
-				)
+					(reference "C50")
+					(unit 1)
+				)

Commit message: done routing!
Connections:
- net GND: now also R33.2; no longer R35.2
- net NTC_FET: now also R33.1, R35.2; no longer R33.2, R35.1
- net VDD: now also R35.1; no longer R33.1
Other:
- moved on the sheet: R33, R35
Changed lines of the file:
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@@
 	(symbol
 		(lib_id "Device:R_US")
-		(at 181.61 91.44 0)
+		(at 181.61 76.2 0)
 		(unit 1)
 		(exclude_from_sim no)
@@
 		(fields_autoplaced yes)
 		(property "Reference" "R35"
-			(at 184.15 90.1699 0)
+			(at 184.15 74.9299 0)
 			(effects
 				(font
@@
 		)
 		(property "Value" "10k NTC"
-			(at 184.15 92.7099 0)
+			(at 184.15 77.4699 0)
 			(effects
 				(font
@@
 		)
 		(property "Footprint" "hn_lib:hn_R_0805"
-			(at 182.626 91.694 90)
+			(at 182.626 76.454 90)
 			(effects
 				(font
@@
 		)
 		(property "Datasheet" "~"
-			(at 181.61 91.44 0)
+			(at 181.61 76.2 0)
 			(effects
 				(font
@@
 		)
 		(property "Description" "Resistor, US symbol"
-			(at 181.61 91.44 0)
+			(at 181.61 76.2 0)
 			(effects
 				(font
@@
 		)
 		(property "part" "Murata NCP21XV103J03RA"
-			(at 181.61 91.44 0)
+			(at 181.61 76.2 0)
 			(effects
 				(font
@@
 	(symbol
 		(lib_id "Device:R_US")
-		(at 181.61 76.2 0)
+		(at 181.61 91.44 0)
 		(unit 1)
 		(exclude_from_sim no)
@@
 		(fields_autoplaced yes)
 		(property "Reference" "R33"
-			(at 184.15 74.9299 0)
+			(at 184.15 90.1699 0)
 			(effects
 				(font
@@
 		)
 		(property "Value" "4.7k"
-			(at 184.15 77.4699 0)
+			(at 184.15 92.7099 0)
 			(effects
 				(font
@@
 		)
 		(property "Footprint" "hn_lib:hn_R_0402"
-			(at 182.626 76.454 90)
+			(at 182.626 91.694 90)
 			(effects
 				(font
@@
 		)
 		(property "Datasheet" "~"
-			(at 181.61 76.2 0)
+			(at 181.61 91.44 0)
 			(effects
 				(font
@@
 		)
 		(property "Description" ""
-			(at 181.61 76.2 0)
+			(at 181.61 91.44 0)
 			(effects
 				(font
@@
 		)
 		(property "part" "YAGEO RC0402JR-074K7L"
-			(at 181.61 76.2 90)
+			(at 181.61 91.44 90)
 			(effects
 				(font
